Commit message: add physical attribute

File: src/neobot_description/urdf/neobot_base.urdf (robot description, URDF)
Before this commit: robot neobot, 7 links, 6 joints
Links:
- link base_link: mass None -> 0.2; geometry collision cylinder length=0.12 radius=0.10; visual cylinder length=0.12 radius=0.10
- link caster_link: mass None -> 0.02; geometry collision sphere radius=0.016; visual sphere radius=0.016
- link imu_link: mass None -> 0.1; geometry collision box size=0.02 0.02 0.02; visual box size=0.02 0.02 0.02
- link laser_link: mass None -> 0.1; geometry collision cylinder length=0.02 radius=0.02; visual cylinder length=0.02 radius=0.02
- link left_wheel_link: mass None -> 0.2; geometry collision cylinder length=0.04 radius=0.032; visual cylinder length=0.04 radius=0.032
- link right_wheel_link: mass None -> 0.2; geometry collision cylinder length=0.04 radius=0.032; visual cylinder length=0.04 radius=0.032
Joints:
- joint caster_joint: axis (none) -> 0 1 0

Commit message: change neobot description

File: src/neobot_description/urdf/neobot_base.urdf (robot description, URDF)
Before this commit: robot neobot, 7 links, 6 joints
Links:
- removed link base_footprint
- link base_link: mass 0.2 -> None; geometry visual cylinder length=0.12 radius=0.10
- link caster_link: mass 0.02 -> None; geometry visual sphere radius=0.016
- link imu_link: mass 0.1 -> None; geometry visual box size=0.02 0.02 0.02
- link laser_link: mass 0.1 -> None; geometry visual cylinder length=0.02 radius=0.02
- link left_wheel_link: mass 0.2 -> None; geometry visual cylinder length=0.04 radius=0.032
- link right_wheel_link: mass 0.2 -> None; geometry visual cylinder length=0.04 radius=0.032
Joints:
- removed joint base_joint
